File: GateDriverBreakoutboard_PMSM_Project/GateDriverBreakoutboard_PMSM_Project.kicad_sch (KiCad schematic)
At the start: 9 parts, among them Q1 IRFB3206, Q2 IRFB3206

Commit message: Added DC in and 3 Phase out connectors to the schematic
Parts:
- added J1: XT30PW-M, Connector_AMASS:AMASS_XT30PW-M_1x02_P2.50mm_Horizontal, symbol Connector_Generic:Conn_01x02
- added J2: MR30PW-FB, Connector_AMASS:AMASS_MR30PW-FB_1x03_P3.50mm_Horizontal, symbol Connector_Generic:Conn_01x03
Connections:
- net GND: now also J1.1 (Pin_1)
- net Vdrive: now also Q1.2 (D), J1.2 (Pin_2)
